Commit message: add lidar

File: ngeeann_av_description/urdf/ngeeann_av.urdf (robot description, URDF)
Before this commit: robot ngeeann_av, 11 links, 10 joints
Links:
- added link lidar, mass 0.01; visual mesh filename=package://ngeeann_av/meshes/VLP16_scan.dae
- added link lidar_base_link, mass 0.83; collision cylinder length=0.0717 radius=0.0516; visual mesh filename=package://ngeeann_av/meshes/VLP16_base_1.dae
- link imu_link: mass None -> 0.1
Joints:
- added joint lidar_base_mount_joint: type fixed, parent base_link, child lidar_base_link, origin xyz=0 0 1.5 rpy=0 0 0
- added joint lidar_base_scan_joint: type fixed, parent lidar_base_link, child lidar, origin xyz=0 0 0.0377 rpy=0 0 0
