Commit message: u

File: ngeeann_av_description/urdf/VLP-16.urdf.xacro (robot description, xacro)
@@ -18,10 +18,10 @@
       <visual>
         <geometry>
-          <mesh filename="package://ngeeann_av/meshes/VLP16_base_1.dae" />
+          <mesh filename="package://ngeeann_av_description/meshes/VLP16_base_1.dae" />
         </geometry>
       </visual>
       <visual>
         <geometry>
-          <mesh filename="package://ngeeann_av/meshes/VLP16_base_2.dae" />
+          <mesh filename="package://ngeeann_av_description/meshes/VLP16_base_2.dae" />
         </geometry>
       </visual>
@@ -47,5 +47,5 @@
         <origin xyz="0 0 -0.0377" />
         <geometry>
-          <mesh filename="package://ngeeann_av/meshes/VLP16_scan.dae" />
+          <mesh filename="package://ngeeann_av_description/meshes/VLP16_scan.dae" />
         </geometry>
       </visual>

File: ngeeann_av_description/urdf/ngeeann_av.urdf (robot description, URDF)
Before this commit: robot ngeeann_av, 13 links, 12 joints
Links:
- removed link hokuyo_link
- removed link spoiler_link
- link lidar: geometry visual mesh filename=package://ngeeann_av_description/meshes/VLP16_scan.dae
- link lidar_base_link: geometry collision cylinder length=0.0717 radius=0.0516; visual mesh filename=package://ngeeann_av_description/meshes/VLP16_base_1.dae
Joints:
- removed joint hokuyo_joint
- removed joint spoiler_joint

File: ngeeann_av_description/urdf/ngeeann_av.xacro (robot description, xacro)
@@ -25,5 +25,5 @@
     <child link="chassis_link"/>
   </joint>
-  <joint name="hokuyo_joint" type="fixed">
+  <!-- <joint name="hokuyo_joint" type="fixed">
     <axis xyz="0 1 0" />
     <origin xyz="0 2.34 0.24" rpy="0 0 1.5708"/>
@@ -49,5 +49,5 @@
       <inertia ixx="1e-6" ixy="0" ixz="0" iyy="1e-6" iyz="0" izz="1e-6" />
     </inertial>
-  </link>
+  </link> -->
   <link name="chassis_link">
     <inertial>
@@ -88,5 +88,5 @@
     <xacro:box_inertia m="0.1" w="0.1" d="0.1" h="0.1"/>
   </link>
-  <joint name="spoiler_joint" type="fixed">
+  <!-- <joint name="spoiler_joint" type="fixed">
     <origin xyz="0 0.05 -0.05" rpy="1.5708 0 3.14159" />
     <parent link="chassis_link"/>
@@ -107,5 +107,5 @@
       </geometry>
     </collision>
-  </link>
+  </link> -->
   <link name="br_1">
     <inertial>
@@ -249,5 +249,5 @@
     <gravity>true</gravity>
   </gazebo>
-  <gazebo reference="spoiler_link">
+  <!-- <gazebo reference="spoiler_link">
     <material>Gazebo/DarkGrey</material>
     <mu1>0.2</mu1>
@@ -255,5 +255,5 @@
     <selfCollide>true</selfCollide>
     <gravity>true</gravity>
-  </gazebo>
+  </gazebo> -->
   <gazebo reference="br_1">
     <material>Gazebo/DarkGrey</material>
@@ -296,4 +296,5 @@
     <plugin filename="libgazebo_ros_imu_sensor.so" name="imu_plugin">
         <ros>
+          <namespace>/ngeeann_av</namespace>
           <remapping>~/out:=imu</remapping>
         </ros>

Commit message: costmap

File: ngeeann_av_description/urdf/VLP-16.urdf.xacro (robot description, xacro)
@@ -2,5 +2,5 @@
 <robot xmlns:xacro="http://www.ros.org/wiki/xacro" name="VLP-16">
   <xacro:property name="M_PI" value="3.1415926535897931" />
-  <xacro:macro name="VLP-16" params="*origin parent:=base_link name:=velodyne topic:=/velodyne_points hz:=10 lasers:=16 samples:=1875 collision_range:=0.3 min_range:=0.9 max_range:=130.0 noise:=0.008 min_angle:=-${M_PI} max_angle:=${M_PI} gpu:=false">
+  <xacro:macro name="VLP-16" params="*origin parent:=base_link name:=velodyne topic:=/points2 hz:=10 lasers:=16 samples:=1875 collision_range:=0.3 min_range:=0.9 max_range:=130.0 noise:=0.008 min_angle:=-${M_PI} max_angle:=${M_PI} gpu:=false">
     <joint name="${name}_base_mount_joint" type="fixed">
       <xacro:insert_block name="origin" />

File: ngeeann_av_description/urdf/ngeeann_av.xacro (robot description, xacro)
@@ -361,5 +361,5 @@
   </gazebo>
   <xacro:include filename="./VLP-16.urdf.xacro"/>
-  <xacro:VLP-16 parent="base_link" name="lidar" topic="/velodyne_points" hz="10" samples="440" gpu="${gpu}">
+  <xacro:VLP-16 parent="base_link" name="lidar" topic="/points2" hz="10" samples="440" gpu="${gpu}">
     <origin xyz="0 0 1.5" rpy="0 0 0" />
   </xacro:VLP-16>

File: velodyne_description/urdf/HDL-32E.urdf.xacro (robot description, xacro)
@@ -2,5 +2,5 @@
 <robot xmlns:xacro="http://www.ros.org/wiki/xacro" name="HDL-32E">
   <xacro:property name="M_PI" value="3.1415926535897931" />
-  <xacro:macro name="HDL-32E" params="*origin parent:=base_link name:=velodyne topic:=/velodyne_points hz:=10 lasers:=32 samples:=2187 collision_range:=0.3 min_range:=0.9 max_range:=130.0 noise:=0.008 min_angle:=-${M_PI} max_angle:=${M_PI} gpu:=false">
+  <xacro:macro name="HDL-32E" params="*origin parent:=base_link name:=velodyne topic:=/points2 hz:=10 lasers:=32 samples:=2187 collision_range:=0.3 min_range:=0.9 max_range:=130.0 noise:=0.008 min_angle:=-${M_PI} max_angle:=${M_PI} gpu:=false">
     <joint name="${name}_base_mount_joint" type="fixed">
       <xacro:insert_block name="origin" />

File: velodyne_description/urdf/VLP-16.urdf.xacro (robot description, xacro)
@@ -2,5 +2,5 @@
 <robot xmlns:xacro="http://www.ros.org/wiki/xacro" name="VLP-16">
   <xacro:property name="M_PI" value="3.1415926535897931" />
-  <xacro:macro name="VLP-16" params="*origin parent:=base_link name:=velodyne topic:=/velodyne_points hz:=10 lasers:=16 samples:=1875 collision_range:=0.3 min_range:=0.9 max_range:=130.0 noise:=0.008 min_angle:=-${M_PI} max_angle:=${M_PI} gpu:=false">
+  <xacro:macro name="VLP-16" params="*origin parent:=base_link name:=velodyne topic:=/points2 hz:=10 lasers:=16 samples:=1875 collision_range:=0.3 min_range:=0.9 max_range:=130.0 noise:=0.008 min_angle:=-${M_PI} max_angle:=${M_PI} gpu:=false">
     <joint name="${name}_base_mount_joint" type="fixed">
       <xacro:insert_block name="origin" />

File: velodyne_description/urdf/example.urdf.xacro (robot description, xacro)
@@ -31,9 +31,9 @@
   </link>
   <xacro:include filename="$(find velodyne_description)/urdf/VLP-16.urdf.xacro"/>
-  <xacro:VLP-16 parent="base_link" name="velodyne" topic="/velodyne_points" hz="10" samples="440" gpu="${gpu}">
+  <xacro:VLP-16 parent="base_link" name="velodyne" topic="/points2" hz="10" samples="440" gpu="${gpu}">
     <origin xyz="0 0 0.4" rpy="0 0 0" />
   </xacro:VLP-16>
   <xacro:include filename="$(find velodyne_description)/urdf/HDL-32E.urdf.xacro"/>
-  <xacro:HDL-32E parent="base_link" name="velodyne2" topic="/velodyne_points2" hz="10" samples="220" gpu="${gpu}">
+  <xacro:HDL-32E parent="base_link" name="velodyne2" topic="/points2" hz="10" samples="220" gpu="${gpu}">
     <origin xyz="0 0 0.6" rpy="0 0 0" />
   </xacro:HDL-32E>
